File: ATMega8-Dev.kicad_pcb (KiCad board)
At the start: 2 copper layers, 55 x 35 mm, 33 parts, among them J1 PORTB, J2 USB_C_Receptacle_USB2.0_16P, J3 PORTC, J4 PORTD, J5 Conn_02x03_Odd_Even, U1 AMS1117-3.3, U2 CP2102-GM, U3 ATmega328-A, Y1 8MHz

Commit message: Page Set
Routing:
- net GND: vias 105 -> 107
Changed lines of the file:
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@@
 	)
 	(paper "A4")
+	(title_block
+		(title "ATMega328A-dev-board")
+		(date "2026-10-04")
+		(rev "V1.0")
+		(company "Luftgekuhlt")
+		(comment 1 "Designed by: Harsha")
+	)
 	(layers
 		(0 "F.Cu" signal)
@@
 	)
 	(setup
+		(stackup
+			(layer "F.SilkS"
+				(type "Top Silk Screen")
+			)
+			(layer "F.Paste"
+				(type "Top Solder Paste")
+			)
+			(layer "F.Mask"
+				(type "Top Solder Mask")
+				(thickness 0.01)
+			)
+			(layer "F.Cu"
+				(type "copper")
+				(thickness 0.035)
+			)
+			(layer "dielectric 1"
+				(type "core")
+				(thickness 1.51)
+				(material "FR4")
+				(epsilon_r 4.5)
+				(loss_tangent 0.02)
+			)
+			(layer "B.Cu"
+				(type "copper")
+				(thickness 0.035)
+			)
+			(layer "B.Mask"
+				(type "Bottom Solder Mask")
+				(thickness 0.01)
+			)
+			(layer "B.Paste"
+				(type "Bottom Solder Paste")
+			)
+			(layer "B.SilkS"
+				(type "Bottom Silk Screen")
+			)
+			(copper_finish "None")
+			(dielectric_constraints no)
+		)
 		(pad_to_mask_clearance 0)
 		(allow_soldermask_bridges_in_footprints no)
@@
 				(font
 					(size 1 1)
-					(thickness 0.15)
+					(thickness 0.2)
+					(bold yes)
 				)
 			)
@@
 		(tags "capacitor handsolder")
 		(property "Reference" "C2"
-			(at 0 -1.68 90)
+			(at -2.9875 0.05 90)
 			(layer "F.SilkS")
 			(effects
@@
 		(tags "Through hole socket strip THT 1x06 2.54mm single row")
 		(property "Reference" "J4"
-			(at 0 -2.77 90)
+			(at 0 -2.5 90)
 			(layer "F.SilkS")
 			(effects
@@
 	)
 	(via
+		(at 164.5 122)
+		(size 0.6)
+		(drill 0.3)
+		(layers "F.Cu" "B.Cu")
+		(net "GND")
+	)
+	(via
 		(at 133.75 94.5)
 		(size 0.6)
@@
 		(size 0.6)
 		(drill 0.3)
+		(layers "F.Cu" "B.Cu")
+		(net "GND")
+	)
+	(via
+		(at 164.5 120.5)
+		(size 0.6)
+		(drill 0.3)
