File: ATMega8-Dev.kicad_sch (KiCad schematic)
At the start: 32 parts, among them J1 PORTB, J2 USB_C_Receptacle_USB2.0_16P, J3 PORTC, J4 PORTD, J5 Conn_02x03_Odd_Even, SW1 RST, U1 AMS1117-3.3, U2 CP2102-GM, U3 ATmega328-A, Y1 8MHz

Commit message: Page Set
Parts:
- J2: value USB_C_Receptacle_USB2.0_16P -> USB_C_16P
- J5: value Conn_02x03_Odd_Even -> ISP Connnector
Other:
- note added: "5V TO 3V3 REGULATOR"
- note added: "CRYSTAL"
- note added: "I2C PULLUPS"
- note added: "ISP PROGRAMMER HEADER"
- note added: "MCU"
- note added: "Reset Button"
- note added: "USB CC RESISTORS"
- note added: "USB RECEPTACLE"
- note added: "USB TO UART BRIDGE"
- company: (none) -> Luftgekuhlt
- title: (none) -> ATMEGA328A-dev-board
- moved on the sheet: C1, C10, C12, C13, C2, C7, C9, J5, R1, R3, R4, U1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
